Commit message: update

File: assets/urdf/ycb/rigid_body/rigid_body.urdf (robot description, URDF)
Before this commit: robot mug, 1 links, 0 joints
Links:
- link mug: geometry collision mesh filename=ycb/rigid_body/table_top.obj scale=1. 1. 1.; visual mesh filename=ycb/rigid_body/table_top.obj scale=1. 1. 1.
