Commit message: start real2sim

File: assets/urdf/ycb/red_cube/red_cube.urdf (robot description, URDF)
Before this commit: robot cube, 1 links, 0 joints
Links:
- link cube: mass 0.102 -> 0.026; geometry collision mesh filename=ycb/red_cube/base.obj scale=0.01 0.01 0.01; visual mesh filename=ycb/red_cube/base.obj scale=0.01 0.01 0.01

Commit message: update

File: assets/urdf/ycb/red_cube/red_cube.urdf (robot description, URDF)
Before this commit: robot cube, 1 links, 0 joints
Links:
- link cube: mass 0.026 -> 0.2; geometry collision mesh filename=ycb/red_cube/base.obj scale=1. 1. 1.; visual mesh filename=ycb/red_cube/base.obj scale=1. 1. 1.
